File: MMS_SSTC/MMS_SSTC.kicad_sch (KiCad schematic)
At the start: 22 parts, among them J2 Screw_Terminal_01x02, Q1 FQA8N100C, U1 NE555P, U2 UCC37322P, Y1 CXO_DIP8

Commit message: Clean up PCB after build test, add heat sink to assembly
Parts:
- TVS1: footprint Diode_THT:D_DO-27_P12.70mm_Horizontal -> Diode_THT:D_DO-15_P10.16mm_Horizontal
Changed lines of the file:
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@@
 			)
 		)
-		(property "Footprint" "Diode_THT:D_DO-27_P12.70mm_Horizontal"
+		(property "Footprint" "Diode_THT:D_DO-15_P10.16mm_Horizontal"
 			(at 152.4 135.89 0)
 			(hide yes)
