File: MMS_SSTC/MMS_SSTC.kicad_sch (KiCad schematic)
At the start: 22 parts, among them J2 Screw_Terminal_01x02, Q1 FQA8N100C, U1 NE555P, U2 UCC37322P, Y1 CXO_DIP8

Commit message: Prepare meshes for production
Parts:
- L1: value 4T:800T -> 4T:700T
Changed lines of the file:
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@@
 			)
 		)
-		(property "Value" "4T:800T"
+		(property "Value" "4T:700T"
 			(at 213.36 132.4609 90)
 			(show_name no)
