File: MMS_SSTC/MMS_SSTC.kicad_pcb (KiCad board)
At the start: 2 copper layers, 80 x 80 mm, 39 parts, among them J1 Screw_Terminal_01x02, J2 Screw_Terminal_01x02, Q1 FQA8N100C, U1 NE555P, U2 UCC37322P, U3 LM7812_TO220, U4 LM7805_TO220, Y1 CXO_DIP8

Commit message: Prepare meshes for production
Changed lines of the file:
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@@
-	)
-	(segment
-		(start 165.24 86.32)
-		(end 161.86 86.32)
-		(width 1)
-		(layer "B.Cu")
-		(net "+12V")
-	)
-	(segment
-		(start 161.86 86.32)
-		(end 161.8 86.26)
-		(width 1)
-		(layer "B.Cu")
-		(net "+12V")
 	)
 	(segment
@@
 		(start 139.55 85.29)
 		(end 141.86 87.6)
+		(width 0.5)
+		(layer "B.Cu")
+		(net "+12V")
+	)
+	(segment
+		(start 165.04 86.32)
+		(end 161.86 86.32)
 		(width 0.5)
 		(layer "B.Cu")
@@
 		(width 0.5)
 		(layer "B.Cu")
+		(net "+12V")
+	)
+	(segment
+		(start 161.86 86.32)
+		(end 161.8 86.26)
+		(width 0.5)
+		(layer "B.Cu")
