File: MMS_SSTC/PSU.kicad_sch (KiCad schematic)
At the start: 18 parts, among them J1 Screw_Terminal_01x02, SW1 SW_SPST, U3 LM7812_TO220, U4 LM7805_TO220

Commit message: Prepare meshes for production
Other:
- note added: "i dont remember why i hate this rectifier"
Changed lines of the file:
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@@
+		)
+	)
+	(text "i dont remember why i hate this rectifier"
+		(exclude_from_sim no)
+		(at 130.048 111.76 0)
+		(effects
+			(font
+				(size 1.27 1.27)
+			)
 		)
 	)
